File: pcb/msp_stuff.kicad_pcb (KiCad board)
At the start: 2 copper layers, 88.9 x 63.5 mm, 24 parts, among them U1 RC1602A-GHW-ESX

Commit message: continued restructuring of repo, commencing the 'pruning' of old branches
Parts:
- removed the REF** at (116.8, 147.3)
- removed the REF** at (124.5, 149.9)
- added REF**: PinSocket_1x01_P2.54mm_Vertical, Connector_PinSocket_2.54mm:PinSocket_1x01_P2.54mm_Vertical, F.Cu at (119.4, 148.6)
- R1, R2, R3: footprint Resistor_SMD:R_0201_0603Metric -> Resistor_SMD:R_1206_3216Metric_Pad1.30x1.75mm_HandSolder
- moved D1 6.57 mm to (90.2, 105.4)
- moved D2 6.57 mm to (90.2, 101.6)
- moved D3 6.57 mm to (90.2, 97.8)
- moved R1 2.76 mm to (99.1, 105.4)
- moved R2 2.76 mm to (99.1, 101.6)
- moved R3 2.76 mm to (99.1, 97.8)
- moved REF** 1.27 mm to (137.2, 105.4)
Connections:
- R1 pad 1: Net-(R1-Pad1) -> Net-(D1-Pad2)
- R1 pad 2: Net-(D1-Pad2) -> Net-(R1-Pad1)
- R2 pad 1: Net-(R2-Pad1) -> Net-(D2-Pad2)
- R2 pad 2: Net-(D2-Pad2) -> Net-(R2-Pad1)
- R3 pad 1: Net-(R3-Pad1) -> Net-(D3-Pad2)
- R3 pad 2: Net-(D3-Pad2) -> Net-(R3-Pad1)
- REF** pad 6: (no net) -> +BATT
- REF** pad 1: GND -> +BATT
Routing:
- net +BATT: track 198.0 -> 263.3 mm, vias 5 -> 1
- net GND: track 280.5 -> 265.1 mm, vias 3 -> 4
- net Net-(R3-Pad1): track 145.4 -> 153.2 mm
- net Net-(R1-Pad1): track 124.3 -> 131.5 mm
- net Net-(R2-Pad1): track 135.4 -> 142.5 mm
- net Net-(D3-Pad2): track 8.97 -> 5.85 mm
- net Net-(D2-Pad2): track 8.97 -> 5.85 mm
- net Net-(D1-Pad2): track 8.97 -> 5.85 mm
Other:
- board text added: "BT EN"
- board text added: "BT VCC"
- board text added: "GND"
- board text added: "LCD Switch"
- board text removed: "BT 3V A"
- board text removed: "BT 3V B"
- board text removed: "BT GND A"
- board text removed: "BT GND B"
- board text removed: "LCD Switch A"
- board text removed: "LCD Switch B"

Commit message: update bluetooth buttons
Parts:
- added REF**: PinSocket_1x01_P2.54mm_Vertical, Connector_PinSocket_2.54mm:PinSocket_1x01_P2.54mm_Vertical, F.Cu at (109.2, 147.3)
- added REF**: PinSocket_1x01_P2.54mm_Vertical, Connector_PinSocket_2.54mm:PinSocket_1x01_P2.54mm_Vertical, F.Cu at (114.3, 149.9)
Routing:
- net +BATT: track 263.3 -> 258.0 mm
Other:
- board text added: "BT EN 1"
- board text added: "BT EN 2"
- board text added: "BT VCC 1"
- board text added: "BT VCC 2"
- board text added: "LCD Switch 1"
- board text added: "LCD Switch 2"
- board text removed: "BT EN"
- board text removed: "BT VCC"
- board text removed: "LCD Switch"

Commit message: fix screen and bluetooth
Connections:
- REF** pad 7: Net-(U1-Pad14) -> (no net)
- REF** pad 7: (no net) -> Net-(U1-Pad14)
- REF** pad 1: (no net) -> +BATT
- REF** pad 2: (no net) -> +BATT
- REF** pad 3: (no net) -> GND
- REF** pad 4: GND -> (no net)
- REF** pad 5: +BATT -> (no net)
- REF** pad 6: +BATT -> (no net)
- REF** pad 1: +BATT -> (no net)
- RV1 pad 1: +BATT -> (no net)
- U1 pad 2: +BATT -> (no net)
Routing:
- net (no net): track 49.6 -> 126.1 mm, vias 0 -> 3
- net +BATT: track 258.0 -> 200.4 mm
- net Net-(U1-Pad14): track 30.7 -> 41.0 mm, vias 0 -> 1
- net Net-(RV1-Pad2): track 41.5 -> 40.2 mm
- net GND: track 265.1 -> 264.1 mm
